File: Electrical/5 - CAD project/BrimEff.sch (EAGLE design)
At the start: 106 parts, among them IC1 CP2101, IC2 74LVC1T45W6-7, J1 455-1750-1-ND, J3 DNI, J5 WM9734TR-ND, J6 PJ-031CCHINA, Q2 FDN306P, Q3 Si2300DS, T1 BC847, T2 BC847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

Commit message: News
Other:
- note added: "47k||1M2 = 45.289k"
Changed lines of the file:
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@@
 and
 screw terminal</text>
+<text x="167.64" y="139.7" size="1.778" layer="97">47k||1M2 = 45.289k</text>
 </plain>
 <instances>
